Commit message: Add most elements to complete scope for #2
Time to clean up!

File: roamr_description/urdf/roamr_robot.urdf.xacro (robot description, xacro)
@@ -3,7 +3,6 @@
   <xacro:include filename="roamr_legwheel.xacro.xml"/>
   <!-- SI Units -->
-  <!-- TODO: Move geometry to YAML file -->
-  <!-- xacro:property name="yaml_file" value="roamr_geometry.yaml" / -->
-  <!-- xacro:property name="geom" value="${load_yaml(yaml_file)}"/ -->
+  <xacro:arg name="geom_file" default="$(find roamr_description)/config/roamr_geometry.yaml" />
+  <xacro:property name="geom" value="${xacro.load_yaml('$(arg geom_file)')}" />
   <!-- Start with the chassis as base_link -->
   <link name="base_link">
@@ -15,12 +14,13 @@
   </link>
   <!-- Add the leg-wheels -->
+  <!-- TODO: Add parameters for remaining legwheel geometry -->
   <xacro:roamr_legwheel parent="base_link" suffix="right">
-    <origin rpy="0.0 0.0 ${-60.0*3.14159/180.0}" xyz="0.058 -0.100 0.0" />
+    <origin rpy="0.0 0.0 ${-pi/3.0}" xyz="${geom['legwheel_xyz']['right']}" />
   </xacro:roamr_legwheel>
   <xacro:roamr_legwheel parent="base_link" suffix="left">
-    <origin rpy="0.0 0.0 ${60.0*3.14159/180.0}" xyz="0.058 0.100 0.0" />
+    <origin rpy="0.0 0.0 ${pi/3.0}" xyz="${geom['legwheel_xyz']['left']}" />
   </xacro:roamr_legwheel>
   <xacro:roamr_legwheel parent="base_link" suffix="back">
-    <origin rpy="0.0 0.0 ${3.14159}" xyz="-0.115 0.0 0.0" />
+    <origin rpy="0.0 0.0 ${pi}" xyz="${geom['legwheel_xyz']['back']}" />
   </xacro:roamr_legwheel>
   <!-- TODO: Add base_footprint for navigation if required -->

Commit message: Add namespace for nodes and frames; Complete parameterization of xacro

File: roamr_description/urdf/roamr_robot.urdf.xacro (robot description, xacro)
@@ -3,8 +3,13 @@
   <xacro:include filename="roamr_legwheel.xacro.xml"/>
   <!-- SI Units -->
+  <xacro:arg name="namespace" default="roamr" />
   <xacro:arg name="geom_file" default="$(find roamr_description)/config/roamr_geometry.yaml" />
+  <xacro:property name="ns" value="'$(arg namespace)'" />
   <xacro:property name="geom" value="${xacro.load_yaml('$(arg geom_file)')}" />
+  <xacro:property name="zc" value="${geom['chassis_elevation']}" />
+  <xacro:property name="rw" value="${geom['wheel_radius']}" />
+  <xacro:property name="ll" value="${geom['leg_length']}" /> <!-- DO NOT use ll in expressions! -->
   <!-- Start with the chassis as base_link -->
-  <link name="base_link">
+  <link name="${ns}_base_link">
     <visual>
       <geometry>
@@ -15,14 +20,20 @@
   <!-- Add the leg-wheels -->
   <!-- TODO: Add parameters for remaining legwheel geometry -->
-  <xacro:roamr_legwheel parent="base_link" suffix="right">
+  <xacro:roamr_legwheel zc="${zc}" rw="${rw}" ll="${ll}" parent="${ns}_base_link" prefix="${ns}" suffix="right">
     <origin rpy="0.0 0.0 ${-pi/3.0}" xyz="${geom['legwheel_xyz']['right']}" />
   </xacro:roamr_legwheel>
-  <xacro:roamr_legwheel parent="base_link" suffix="left">
+  <xacro:roamr_legwheel zc="${zc}" rw="${rw}" ll="${ll}" parent="${ns}_base_link" prefix="${ns}" suffix="left">
     <origin rpy="0.0 0.0 ${pi/3.0}" xyz="${geom['legwheel_xyz']['left']}" />
   </xacro:roamr_legwheel>
-  <xacro:roamr_legwheel parent="base_link" suffix="back">
+  <xacro:roamr_legwheel zc="${zc}" rw="${rw}" ll="${ll}" parent="${ns}_base_link" prefix="${ns}" suffix="back">
     <origin rpy="0.0 0.0 ${pi}" xyz="${geom['legwheel_xyz']['back']}" />
   </xacro:roamr_legwheel>
   <!-- TODO: Add base_footprint for navigation if required -->
+  <link name="${ns}_base_footprint" />
+  <joint name="${ns}_base_footprint_joint" type="fixed">
+    <parent link="${ns}_base_link" />
+    <child link="${ns}_base_footprint" />
+    <origin rpy="0 0 0" xyz="0 0 -${zc}" />
+  </joint>
   <!-- TODO: Add dynamic properties for dynamic simulation if required -->
 </robot>

Commit message: Clean up xacro files

File: roamr_description/urdf/roamr_robot.urdf.xacro (robot description, xacro)
@@ -9,5 +9,5 @@
   <xacro:property name="zc" value="${geom['chassis_elevation']}" />
   <xacro:property name="rw" value="${geom['wheel_radius']}" />
-  <xacro:property name="ll" value="${geom['leg_length']}" /> <!-- DO NOT use ll in expressions! -->
+  <xacro:property name="ll" value="${geom['leg_length']}" />
   <!-- Start with the chassis as base_link -->
   <link name="${ns}_base_link">
@@ -19,5 +19,4 @@
   </link>
   <!-- Add the leg-wheels -->
-  <!-- TODO: Add parameters for remaining legwheel geometry -->
   <xacro:roamr_legwheel zc="${zc}" rw="${rw}" ll="${ll}" parent="${ns}_base_link" prefix="${ns}" suffix="right">
     <origin rpy="0.0 0.0 ${-pi/3.0}" xyz="${geom['legwheel_xyz']['right']}" />
@@ -29,5 +28,4 @@
     <origin rpy="0.0 0.0 ${pi}" xyz="${geom['legwheel_xyz']['back']}" />
   </xacro:roamr_legwheel>
-  <!-- TODO: Add base_footprint for navigation if required -->
   <link name="${ns}_base_footprint" />
   <joint name="${ns}_base_footprint_joint" type="fixed">

Commit message: Integrate YAML dimensions between FreeCAD macro and roamr_description
- Includes changins a couple dimensions and URDF calculations
- Uses symlink between subdirectories; Could do something fancier on the FreeCAD side, but shouldn't be needed.

File: roamr_description/urdf/roamr_robot.urdf.xacro (robot description, xacro)
@@ -7,5 +7,5 @@
   <xacro:property name="ns" value="'$(arg namespace)'" />
   <xacro:property name="geom" value="${xacro.load_yaml('$(arg geom_file)')}" />
-  <xacro:property name="zc" value="${geom['chassis_elevation']}" />
+  <xacro:property name="zc" value="${geom['wheel_radius'] + geom['caster_height']}" />
   <xacro:property name="rw" value="${geom['wheel_radius']}" />
   <xacro:property name="ll" value="${geom['leg_length']}" />
@@ -18,13 +18,20 @@
     </visual>
   </link>
+  <xacro:macro name="calculate_legwheel_origin" params="angle">
+    <!-- Here, radius is the distance from center of chassis to vertex -->
+    <xacro:property name="radius" value="${geom['chassis_side_length'] / sqrt(3)}" />
+    <xacro:property name="x" value="${radius * cos(angle)}" />
+    <xacro:property name="y" value="${radius * sin(angle)}" />
+    <origin rpy="0.0 0.0 ${angle}" xyz="${x} ${y} 0.0" />
+  </xacro:macro>
   <!-- Add the leg-wheels -->
   <xacro:roamr_legwheel zc="${zc}" rw="${rw}" ll="${ll}" parent="${ns}_base_link" prefix="${ns}" suffix="right">
-    <origin rpy="0.0 0.0 ${-pi/3.0}" xyz="${geom['legwheel_xyz']['right']}" />
+    <xacro:calculate_legwheel_origin angle="${-pi/3.0}" />
   </xacro:roamr_legwheel>
   <xacro:roamr_legwheel zc="${zc}" rw="${rw}" ll="${ll}" parent="${ns}_base_link" prefix="${ns}" suffix="left">
-    <origin rpy="0.0 0.0 ${pi/3.0}" xyz="${geom['legwheel_xyz']['left']}" />
+    <xacro:calculate_legwheel_origin angle="${pi/3.0}" />
   </xacro:roamr_legwheel>
   <xacro:roamr_legwheel zc="${zc}" rw="${rw}" ll="${ll}" parent="${ns}_base_link" prefix="${ns}" suffix="back">
-    <origin rpy="0.0 0.0 ${pi}" xyz="${geom['legwheel_xyz']['back']}" />
+    <xacro:calculate_legwheel_origin angle="${pi}" />
   </xacro:roamr_legwheel>
   <link name="${ns}_base_footprint" />
